File: PCRuler_KiCad/PCRuler_KiCad.kicad_pcb (KiCad board)
At the start: 2 copper layers, 250 x 25 mm, 30 parts, among them Q1 DMMT5401, SW1 CK_KMS2xxG, SW2 CK_KMS2xxG, U1 ICM7555xB, U2 ATmega8-16A, U3 PAM8406D, Y1 Crystal

Commit message: Done design
Parts:
- moved R2 121.2 mm to (233.5, 152.8), turned to -90 degrees
- moved R1 121.0 mm to (233.5, 150.4), turned to -90 degrees
- moved D1 89.3 mm to (171.3, 156.4)
- moved R3 79.7 mm to (174.8, 156.3)
- moved D2 71.5 mm to (147.9, 153.1), turned to 90 degrees
- moved R6 64.7 mm to (140.4, 149.8), turned to -90 degrees
- moved R7 62.4 mm to (136.7, 149.7), turned to -90 degrees
- moved R8 60.2 mm to (132.8, 149.6), turned to -90 degrees
- moved R4 40.5 mm to (147.9, 149.6), turned to -90 degrees
- moved C2 11.3 mm to (180.3, 159.9), turned to 0 degrees
- turned R10 to -90 degrees
Routing:
- net Net-(D2-K): track 0.00 -> 230.5 mm, vias 0 -> 8
- net Net-(U1-DIS): track 0.00 -> 216.8 mm, vias 0 -> 15
- net Net-(Q1A-E1): track 0.00 -> 204.4 mm, vias 0 -> 3
- net Net-(D1-K): track 0.00 -> 196.8 mm, vias 0 -> 7
- net /bus_5: track 0.00 -> 126.0 mm, vias 0 -> 2
- net /bus_4: track 0.00 -> 122.0 mm, vias 0 -> 2
- net Net-(U2-PB1): track 0.00 -> 118.6 mm, vias 0 -> 3
- net /bus_3: track 0.00 -> 118.3 mm, vias 0 -> 2
- net Net-(D1-A): track 0.00 -> 118.0 mm, vias 0 -> 2
- net /bus_2: track 0.00 -> 115.4 mm, vias 0 -> 2
- net /bus_1: track 0.00 -> 109.3 mm
- net Net-(U2-PD2): track 0.00 -> 85.2 mm, vias 0 -> 2
- net Net-(U2-PD1): track 0.00 -> 81.4 mm, vias 0 -> 2
- net Net-(U2-PD3): track 0.00 -> 78.6 mm, vias 0 -> 4
- net Net-(U2-PD4): track 0.00 -> 75.7 mm, vias 0 -> 8
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
Commit message: Re-did almost everything
Parts:
- removed C1, C2, C3, C4, C5: C, Capacitor_SMD:C_1812_4532Metric
- removed D1, D2, D3, D4, D5, D6, D7, D8: LED, LED_SMD:LED_0805_2012Metric
- removed Q1: DMMT5401, Package_TO_SOT_SMD:SOT-23-6
- removed R1, R10, R2, R3, R4, R5, R6, R7, R8, R9: R, Resistor_SMD:R_0402_1005Metric
- removed SW1, SW2: CK_KMS2xxG, Button_Switch_SMD:SW_SPST_CK_KMS2xxGP
- removed U1: ICM7555xB, Package_SO:SOIC-8_3.9x4.9mm_P1.27mm
- removed U2: ATmega8-16A, Package_QFP:TQFP-32_7x7mm_P0.8mm
- removed U3: PAM8406D, Package_SO:SOIC-16_3.9x9.9mm_P1.27mm
- removed Y1: Crystal, Crystal:Crystal_SMD_0603-4Pin_6.0x3.5mm
Routing:
- net Net-(D2-K): track 230.5 -> 0.00 mm, vias 8 -> 0
- net Net-(U1-DIS): track 216.8 -> 0.00 mm, vias 15 -> 0
- net Net-(Q1A-E1): track 204.4 -> 0.00 mm, vias 3 -> 0
- net Net-(D1-K): track 196.8 -> 0.00 mm, vias 7 -> 0
- net /bus_5: track 126.0 -> 0.00 mm, vias 2 -> 0
- net /bus_4: track 122.0 -> 0.00 mm, vias 2 -> 0
- net Net-(U2-PB1): track 118.6 -> 0.00 mm, vias 3 -> 0
- net /bus_3: track 118.3 -> 0.00 mm, vias 2 -> 0
- net Net-(D1-A): track 118.0 -> 0.00 mm, vias 2 -> 0
- net /bus_2: track 115.4 -> 0.00 mm, vias 2 -> 0
- net /bus_1: track 109.3 -> 0.00 mm
- net Net-(U2-PD2): track 85.2 -> 0.00 mm, vias 2 -> 0
- net Net-(U2-PD1): track 81.4 -> 0.00 mm, vias 2 -> 0
- net Net-(U2-PD3): track 78.6 -> 0.00 mm, vias 4 -> 0
- net Net-(U2-PD4): track 75.7 -> 0.00 mm, vias 8 -> 0
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Other:
- board text added: "1"
- board text added: "10 11"
- board text added: "12 13"
- board text added: "14 15"
- board text added: "16 17"
- board text added: "18 19"
- board text added: "2"
- board text added: "20 21"
- board text added: "22 23"
- board text added: "24"
- board text added: "3"
- board text added: "4 5"
- board text added: "6 7"
- board text added: "8 9"

Commit message: Finished layout
Finished layout and added gerbers
Parts:
- added BT1: Battery_Cell, footprints:CONN_TSM-102-01-T-SH_SAI, F.Cu at (250.5, 150.0)
- added D1: LED, LED_SMD:LED_0805_2012Metric, F.Cu at (332.9, 154.2)
- added D10: Inolux_IN-PI554FCH, LED_SMD:LED_Inolux_IN-PI554FCH_PLCC4_5.0x5.0mm_P3.2mm, F.Cu at (104.0, 159.0)
- added D11: Inolux_IN-PI554FCH, LED_SMD:LED_Inolux_IN-PI554FCH_PLCC4_5.0x5.0mm_P3.2mm, F.Cu at (114.0, 159.0)
- added D12: Inolux_IN-PI554FCH, LED_SMD:LED_Inolux_IN-PI554FCH_PLCC4_5.0x5.0mm_P3.2mm, F.Cu at (124.0, 159.0)
- added D13: Inolux_IN-PI554FCH, LED_SMD:LED_Inolux_IN-PI554FCH_PLCC4_5.0x5.0mm_P3.2mm, F.Cu at (134.0, 159.0)
- added D14: Inolux_IN-PI554FCH, LED_SMD:LED_Inolux_IN-PI554FCH_PLCC4_5.0x5.0mm_P3.2mm, F.Cu at (144.0, 159.0)
- added D15: Inolux_IN-PI554FCH, LED_SMD:LED_Inolux_IN-PI554FCH_PLCC4_5.0x5.0mm_P3.2mm, F.Cu at (154.0, 159.0)
- added D16: Inolux_IN-PI554FCH, LED_SMD:LED_Inolux_IN-PI554FCH_PLCC4_5.0x5.0mm_P3.2mm, F.Cu at (164.0, 159.0)
- added D17: Inolux_IN-PI554FCH, LED_SMD:LED_Inolux_IN-PI554FCH_PLCC4_5.0x5.0mm_P3.2mm, F.Cu at (174.0, 159.0)
- added D18: Inolux_IN-PI554FCH, LED_SMD:LED_Inolux_IN-PI554FCH_PLCC4_5.0x5.0mm_P3.2mm, F.Cu at (184.0, 159.0)
- added D19: Inolux_IN-PI554FCH, LED_SMD:LED_Inolux_IN-PI554FCH_PLCC4_5.0x5.0mm_P3.2mm, F.Cu at (194.0, 159.0)
- added D2: Inolux_IN-PI554FCH, LED_SMD:LED_Inolux_IN-PI554FCH_PLCC4_5.0x5.0mm_P3.2mm, F.Cu at (24.0, 159.0)
- added D20: Inolux_IN-PI554FCH, LED_SMD:LED_Inolux_IN-PI554FCH_PLCC4_5.0x5.0mm_P3.2mm, F.Cu at (204.0, 159.0)
- added D21: Inolux_IN-PI554FCH, LED_SMD:LED_Inolux_IN-PI554FCH_PLCC4_5.0x5.0mm_P3.2mm, F.Cu at (214.0, 159.0)
- added D22: Inolux_IN-PI554FCH, LED_SMD:LED_Inolux_IN-PI554FCH_PLCC4_5.0x5.0mm_P3.2mm, F.Cu at (224.0, 159.0)
- added D23: Inolux_IN-PI554FCH, LED_SMD:LED_Inolux_IN-PI554FCH_PLCC4_5.0x5.0mm_P3.2mm, F.Cu at (234.0, 158.9)
- added D24: Inolux_IN-PI554FCH, LED_SMD:LED_Inolux_IN-PI554FCH_PLCC4_5.0x5.0mm_P3.2mm, F.Cu at (244.0, 159.0)
- added D25: Inolux_IN-PI554FCH, LED_SMD:LED_Inolux_IN-PI554FCH_PLCC4_5.0x5.0mm_P3.2mm, F.Cu at (254.0, 159.0)
- added D3: Inolux_IN-PI554FCH, LED_SMD:LED_Inolux_IN-PI554FCH_PLCC4_5.0x5.0mm_P3.2mm, F.Cu at (34.0, 159.0)
- added D4: Inolux_IN-PI554FCH, LED_SMD:LED_Inolux_IN-PI554FCH_PLCC4_5.0x5.0mm_P3.2mm, F.Cu at (44.0, 159.0)
- added D5: Inolux_IN-PI554FCH, LED_SMD:LED_Inolux_IN-PI554FCH_PLCC4_5.0x5.0mm_P3.2mm, F.Cu at (54.0, 159.0)
- added D6: Inolux_IN-PI554FCH, LED_SMD:LED_Inolux_IN-PI554FCH_PLCC4_5.0x5.0mm_P3.2mm, F.Cu at (64.0, 159.0)
- added D7: Inolux_IN-PI554FCH, LED_SMD:LED_Inolux_IN-PI554FCH_PLCC4_5.0x5.0mm_P3.2mm, F.Cu at (74.0, 159.0)
- added D8: Inolux_IN-PI554FCH, LED_SMD:LED_Inolux_IN-PI554FCH_PLCC4_5.0x5.0mm_P3.2mm, F.Cu at (84.0, 159.0)
- added D9: Inolux_IN-PI554FCH, LED_SMD:LED_Inolux_IN-PI554FCH_PLCC4_5.0x5.0mm_P3.2mm, F.Cu at (94.0, 159.0)
- added J2: USB_C_Receptacle_USB2.0_14P, Connector_USB:USB_C_Receptacle_GCT_USB4110, F.Cu at (331.2, 163.1)
- added J3: Conn_01x04_Pin, Connector_PinSocket_2.54mm:PinSocket_1x04_P2.54mm_Vertical_SMD_Pin1Left, F.Cu at (186.0, 150.2)
- added R1: 10k, Resistor_SMD:R_0402_1005Metric, F.Cu at (211.3, 154.7)
- added R2: 10k, Resistor_SMD:R_0402_1005Metric, F.Cu at (54.1, 152.5)
- added R3: 10k, Resistor_SMD:R_0402_1005Metric, F.Cu at (197.1, 149.1)
- added R4: 470, Resistor_SMD:R_0402_1005Metric, F.Cu at (329.6, 155.8)
- added R5: 10k, Resistor_SMD:R_0402_1005Metric, F.Cu at (40.7, 154.8)
- added R6: 10k, Resistor_SMD:R_0402_1005Metric, F.Cu at (22.0, 154.9)
- added R7: 2k, Resistor_SMD:R_0402_1005Metric, F.Cu at (265.9, 149.6)
- added SW1: SW_DPST, footprints:B3FS-100_OMR, F.Cu at (215.8, 150.3)
- added SW2: SW_DPST, footprints:B3FS-100_OMR, F.Cu at (46.9, 150.5)
- added SW3: SW_DPST, footprints:B3FS-100_OMR, F.Cu at (36.4, 150.5)
- added SW4: SW_DPST, footprints:B3FS-100_OMR, F.Cu at (205.2, 150.3)
- added SW5: SW_DPST, footprints:B3FS-100_OMR, F.Cu at (25.9, 150.5)
- added SW6: SW_SPDT, footprints:SW_JS102011SCQN, F.Cu at (237.9, 150.8)
- added U1: ESP32-C6-MINI-1, RF_Module:ESP32-C6-MINI-1, F.Cu at (315.5, 158.0)
- added U2: MCP73831-2-OT, Package_TO_SOT_SMD:SOT-23-5, F.Cu at (261.2, 150.0)
- added U3: AZ1117CH2-3.3, Package_TO_SOT_SMD:SOT-223-3_TabPin2, F.Cu at (224.7, 150.8)
Routing:
- net GND: track 0.00 -> 526.8 mm, vias 0 -> 4
- net +3.3V: track 0.00 -> 424.7 mm, vias 0 -> 8
- net /BTN_3: track 0.00 -> 338.8 mm, vias 0 -> 12
- net /BTN_2: track 0.00 -> 329.5 mm, vias 0 -> 10
- net /BTN_1: track 0.00 -> 315.6 mm, vias 0 -> 8
- net /LED_DATA: track 0.00 -> 311.0 mm, vias 0 -> 2
- net Net-(J3-Pin_2): track 0.00 -> 177.5 mm, vias 0 -> 10
- net Net-(J3-Pin_1): track 0.00 -> 137.0 mm, vias 0 -> 8
- net /BOOT: track 0.00 -> 134.8 mm, vias 0 -> 4
- net /RESET: track 0.00 -> 121.0 mm, vias 0 -> 6
- net +5V: track 0.00 -> 91.0 mm, vias 0 -> 2
- net /charger_status: track 0.00 -> 81.1 mm, vias 0 -> 2
- net +BATT: track 0.00 -> 25.1 mm
- net /USB_D-: track 0.00 -> 19.4 mm, vias 0 -> 2
- net /USB_D+: track 0.00 -> 18.3 mm, vias 0 -> 2
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Other:
- board size 250 x 25 mm -> 314.9 x 23.5 mm
