File: PCRuler_KiCad/PCRuler_KiCad.kicad_sch (KiCad schematic)
At the start: 30 parts, among them Q1 DMMT5401, SW1 CK_KMS2xxG, SW2 CK_KMS2xxG, U1 ICM7555xB, U2 ATmega8-16A, U3 PAM8406D, Y1 Crystal

Commit message: Re-did almost everything
Parts:
- removed C1, C2, C3, C4, C5: C, Capacitor_SMD:C_1812_4532Metric, symbol Device:C
- removed D1, D2, D3, D4, D5, D6, D7, D8: LED, LED_SMD:LED_0805_2012Metric, symbol Device:LED
- removed Q1: DMMT5401, Package_TO_SOT_SMD:SOT-23-6, symbol Transistor_BJT:DMMT5401
- removed R1, R10, R2, R3, R4, R5, R6, R7, R8, R9: R, Resistor_SMD:R_0402_1005Metric, symbol Device:R
- removed SW1, SW2: CK_KMS2xxG, Button_Switch_SMD:SW_SPST_CK_KMS2xxGP, symbol Switch:CK_KMS2xxG
- removed U1: ICM7555xB, Package_SO:SOIC-8_3.9x4.9mm_P1.27mm, symbol Timer:ICM7555xB
- removed U2: ATmega8-16A, Package_QFP:TQFP-32_7x7mm_P0.8mm, symbol MCU_Microchip_ATmega:ATmega8-16A
- removed U3: PAM8406D, Package_SO:SOIC-16_3.9x9.9mm_P1.27mm, symbol Amplifier_Audio:PAM8406D
- removed Y1: Crystal, Crystal:Crystal_SMD_0603-4Pin_6.0x3.5mm, symbol Device:Crystal
- added D1, D10, D11, D12, D13, D14, D15, D16, D17, D18, D19, D2, D20, D21, D22, D23, D24, D3, D4, D5, D6, D7, D8, D9: Inolux_IN-PI554FCH, LED_SMD:LED_Inolux_IN-PI554FCH_PLCC4_5.0x5.0mm_P3.2mm, symbol LED:Inolux_IN-PI554FCH
- added J1: USB_C_Receptacle_USB2.0_14P, symbol Connector:USB_C_Receptacle_USB2.0_14P
- added U1: ESP32-C6-MINI-1, RF_Module:ESP32-C6-MINI-1, symbol RF_Module:ESP32-C6-MINI-1
Connections:
- new net: D22.4 (DO), D23.2 (DIN)
- new net: D17.3 (VDD), D18.3 (VDD), D19.3 (VDD), D20.3 (VDD), D21.3 (VDD), D22.3 (VDD), D23.3 (VDD), D24.3 (VDD)
- new net: D23.4 (DO), D24.2 (DIN)
- new net: D18.4 (DO), D19.2 (DIN)
- new net: D19.4 (DO), D20.2 (DIN)
- new net: D1.1 (VSS), D2.1 (VSS), D3.1 (VSS), D4.1 (VSS), D5.1 (VSS), D6.1 (VSS), D7.1 (VSS), D8.1 (VSS)
- new net: D1.4 (DO), D2.2 (DIN)
- new net: D2.4 (DO), D3.2 (DIN)
- new net: D21.4 (DO), D22.2 (DIN)
- new net: D20.4 (DO), D21.2 (DIN)
- new net: D7.4 (DO), D8.2 (DIN)
- new net: D8.4 (DO), D9.2 (DIN)
- new net: D3.4 (DO), D4.2 (DIN)
- new net: D4.4 (DO), D5.2 (DIN)
- new net: J1.A1 (GND), J1.A12 (GND), J1.B1 (GND), J1.B12 (GND), J1.S1 (SHIELD)
- new net: J1.A6 (D+), J1.B6 (D+)
- new net: J1.A7 (D-), J1.B7 (D-)
- new net: D6.4 (DO), D7.2 (DIN)
- new net: D17.4 (DO), D18.2 (DIN)
- new net: D10.1 (VSS), D11.1 (VSS), D12.1 (VSS), D13.1 (VSS), D14.1 (VSS), D15.1 (VSS), D16.1 (VSS), D9.1 (VSS)
- new net: D13.4 (DO), D14.2 (DIN)
- new net: D10.3 (VDD), D11.3 (VDD), D12.3 (VDD), D13.3 (VDD), D14.3 (VDD), D15.3 (VDD), D16.3 (VDD), D9.3 (VDD)
- new net: D14.4 (DO), D15.2 (DIN)
- new net: D10.2 (DIN), D9.4 (DO)
- new net: D5.4 (DO), D6.2 (DIN)
- new net: D15.4 (DO), D16.2 (DIN)
- new net: D12.4 (DO), D13.2 (DIN)
- new net: D10.4 (DO), D11.2 (DIN)
- new net: D11.4 (DO), D12.2 (DIN)
- new net: U1.1 (GND), U1.11 (GND), U1.14 (GND), U1.2 (GND), U1.36 (GND), U1.37 (GND), U1.38 (GND), U1.39 (GND), U1.40 (GND), U1.41 (GND), U1.42 (GND), U1.43 (GND), U1.44 (GND), U1.45 (GND), U1.46 (GND), U1.47 (GND), U1.48 (GND), U1.49 (GND), U1.50 (GND), U1.51 (GND), U1.52 (GND), U1.53 (GND)
- new net: D16.4 (DO), D17.2 (DIN)
- new net +3.3V: D1.3 (VDD), D2.3 (VDD), D3.3 (VDD), D4.3 (VDD), D5.3 (VDD), D6.3 (VDD), D7.3 (VDD), D8.3 (VDD)
- new net +5V: J1.A4 (VBUS), J1.A9 (VBUS), J1.B4 (VBUS), J1.B9 (VBUS)
- new net GND: D17.1 (VSS), D18.1 (VSS), D19.1 (VSS), D20.1 (VSS), D21.1 (VSS), D22.1 (VSS), D23.1 (VSS), D24.1 (VSS)
- no-connect marks 0 -> 3

Commit message: Finished layout
Finished layout and added gerbers
Parts:
- added BT1: Battery_Cell, footprints:CONN_TSM-102-01-T-SH_SAI, symbol Device:Battery_Cell
- added D1: LED, LED_SMD:LED_0805_2012Metric, symbol Device:LED
- added J2: Conn_01x04_Pin, Connector_PinSocket_2.54mm:PinSocket_1x04_P2.54mm_Vertical_SMD_Pin1Left, symbol Connector:Conn_01x04_Pin
- added J3: Conn_01x02_Pin, Connector_PinSocket_2.54mm:PinSocket_1x02_P2.54mm_Vertical_SMD_Pin1Left, symbol Connector:Conn_01x02_Pin
- added R1: 2k, Resistor_SMD:R_0402_1005Metric, symbol Device:R
- added R2: 470, Resistor_SMD:R_0402_1005Metric, symbol Device:R
- added R3, R4, R5, R6, R7: 10k, Resistor_SMD:R_0402_1005Metric, symbol Device:R
- added SW1, SW2, SW3, SW4, SW5: SW_DPST, footprints:B3FS-100_OMR, symbol Switch:SW_DPST
- added SW6: SW_SPDT, footprints:SW_JS102011SCQN, symbol Switch:SW_SPDT
- added U1: AZ1117CH2-3.3, Package_TO_SOT_SMD:SOT-223-3_TabPin2, symbol Regulator_Linear:AZ1117CH2-3.3
- added U2: MCP73831-2-OT, Package_TO_SOT_SMD:SOT-23-5, symbol Battery_Management:MCP73831-2-OT
- J1: footprint (none) -> Connector_USB:USB_C_Receptacle_GCT_USB4110
- renumbered D19 to D10, D4 to D11, D20 to D13, D5 to D14, D13 to D15, D21 to D16, D6 to D17, D14 to D18, D22 to D19, D1 to D2, D7 to D20, D15 to D21, D23 to D22, D8 to D23, D16 to D24, D24 to D25, D9 to D3, D17 to D4, D2 to D5, D10 to D6, D18 to D7, D3 to D8, D11 to D9, U1 to U3
Connections:
- net +3.3V: now also D10.3 (VDD), D12.3 (VDD), D13.3 (VDD), D15.3 (VDD), D16.3 (VDD), D18.3 (VDD), D19.3 (VDD), D21.3 (VDD), D22.3 (VDD), D24.3 (VDD), D25.3 (VDD), D3.3 (VDD), D4.3 (VDD), D6.3 (VDD), D7.3 (VDD), D9.3 (VDD), U3.3 (3V3), R3.1, R4.1, SW3.1, SW3.2, SW4.1, SW4.2, SW5.1, SW5.2, U1.3 (OUT)
- net +5V: now also R2.1, U2.4 (V_{DD})
- net GND: now also D11.1 (VSS), D12.1 (VSS), D14.1 (VSS), D15.1 (VSS), D17.1 (VSS), D18.1 (VSS), D2.1 (VSS), D20.1 (VSS), D21.1 (VSS), D23.1 (VSS), D24.1 (VSS), D3.1 (VSS), D5.1 (VSS), D6.1 (VSS), D8.1 (VSS), D9.1 (VSS), J1.A1 (GND), J1.A12 (GND), J1.B1 (GND), J1.B12 (GND), J1.S1 (SHIELD), U3.1 (GND), U3.11 (GND), U3.14 (GND), U3.2 (GND), U3.36 (GND), U3.37 (GND), U3.38 (GND), U3.39 (GND), U3.40 (GND), U3.41 (GND), U3.42 (GND), U3.43 (GND), U3.44 (GND), U3.45 (GND), U3.46 (GND), U3.47 (GND), U3.48 (GND), U3.49 (GND), U3.50 (GND), U3.51 (GND), U3.52 (GND), U3.53 (GND), BT1.2 (-), R1.2, R5.2, R6.2, R7.2, SW1.3, SW1.4, SW2.3, SW2.4, U1.2 (GND), U2.2 (V_{SS})
- net USB_D+: now reaches J1.A6 (D+), J1.B6 (D+)
- net USB_D+: now also U3.18 (IO13)
- net USB_D-: now reaches J1.A7 (D-), J1.B7 (D-)
- net USB_D-: now also U3.17 (IO12)
- net LED_DATA: now reaches D2.2 (DIN)
- net LED_DATA: now also U3.24 (IO18)
- net at U3.16 (IO7): now also J2.1 (Pin_1)
- net at U3.22 (IO8): now also J2.2 (Pin_2)
- net BOOT: now reaches U3.23 (IO9)
- net BOOT: now also R4.2, SW2.1, SW2.2
- net BTN_1: now reaches U3.25 (IO19)
- net BTN_1: now also R5.1, SW3.3, SW3.4
- net BTN_2: now reaches U3.26 (IO20)
- net BTN_2: now also R6.1, SW4.3, SW4.4
- net BTN_3: now reaches U3.27 (IO21)
- net BTN_3: now also R7.1, SW5.3, SW5.4
- net at U3.28 (IO22): now also J2.4 (Pin_4)
- net at U3.29 (IO23): now also J2.3 (Pin_3)
- net RX: now reaches U3.30 (RXD0)
- net RX: now also J3.1 (Pin_1)
- net TX: now reaches U3.31 (TXD0)
- net TX: now also J3.2 (Pin_2)
- net RESET: now reaches U3.8 (EN)
- net RESET: now also R3.2, SW1.1, SW1.2
- new net: D1.2 (A), R2.2
- new net: SW6.1 (A), U1.1 (IN)
- new net: R1.1, U2.5 (PROG)
- new net +BATT: BT1.1 (+), SW6.2 (B), U2.3 (V_{BAT})
- new net charger_status: D1.1 (K), U2.1 (STAT)
- no-connect marks 3 -> 13
Other:
- moved on the sheet: U3

Commit message: Added CC resistors
added USB C current declaration resistors
Parts:
- renumbered D3 to D10, D6 to D11, D9 to D12, D12 to D13, D15 to D14, D18 to D15, D21 to D16, D24 to D17, D4 to D18, D7 to D19, D10 to D20, D13 to D21, D16 to D22, D19 to D23, D22 to D24, D5 to D3, D8 to D4, D11 to D5, D14 to D6, D17 to D7, D20 to D8, D23 to D9, J3 to J1, J1 to J2, J2 to J3, R3 to R1, R5 to R2, R4 to R3, R2 to R4, R6 to R5, R7 to R6, R1 to R7, SW3 to SW2, SW4 to SW3, SW2 to SW4, U3 to U1, U1 to U3

Commit message: Fixed USBc
again
Parts:
- added R8, R9: 33k, Resistor_SMD:R_0402_1005Metric, symbol Device:R
Connections:
- net GND: now also R8.2, R9.2
- net at J2.A5 (CC1): now also R9.1
- net at J2.B5 (CC2): now also R8.1
- no-connect marks 13 -> 11
